Commit message: add cmd_vel for nav2 && visual_odom_publisher

File: install/my_robot_description/share/my_robot_description/urdf/my_robot.urdf.xacro (robot description, xacro)
@@ -1 +1,36 @@
-/home/khemin/ros2_ws/src/my_robot_description/urdf/my_robot.urdf.xacro
+<?xml version="1.0"?>
+<robot xmlns:xacro="http://ros.org/wiki/xacro" name="my_robot">
+  <!-- Material definitions -->
+  <material name="blue">
+    <color rgba="0 0 1 1"/>
+  </material>
+  <material name="red">
+    <color rgba="1 0 0 1"/>
+  </material>
+  <!-- Base Link -->
+  <link name="base_link">
+    <visual>
+      <geometry>
+        <box size="0.5 0.5 0.1"/>
+      </geometry>
+      <material name="blue"/>
+    </visual>
+  </link>
+  <!-- Laser Link -->
+  <link name="laser">
+    <visual>
+      <geometry>
+        <cylinder length="0.1" radius="0.05"/>
+      </geometry>
+      <material name="red"/>
+    </visual>
+  </link>
+  <!-- Joint between base_link and laser -->
+  <joint name="laser_joint" type="revolute">
+    <parent link="base_link"/>
+    <child link="laser"/>
+    <origin xyz="0 0 0.1" rpy="0 0 0"/>
+    <axis xyz="0 0 1"/>
+    <limit lower="-1.57" upper="1.57" effort="1.0" velocity="1.0"/>
+  </joint>
+</robot>
